File: kicad files/Nueva carpeta.sch (KiCad schematic (older format))
At the start: 24 parts, among them P1 Power, P2 Analog, P3 Digital, P4 Digital, P5 CONN_01X01, P6 CONN_01X01, P7 CONN_01X01, P8 CONN_01X01, SW1 RESET, U1 ATMEGA328P-PU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

Commit message: agregando .gitignore
Parts:
- C1, C2: symbol device:C -> Nueva-carpeta-rescue:C-device
- D1, D2, D3, D4, D5: symbol device:LED_ALT -> Nueva-carpeta-rescue:LED_ALT-device
- R1, R2, R3, R4, R5, R6: symbol device:R -> Nueva-carpeta-rescue:R-device
- U1: symbol atmel:ATMEGA328P-PU -> Nueva-carpeta-rescue:ATMEGA328P-PU-atmel
- Y1: symbol device:Crystal -> Nueva-carpeta-rescue:Crystal-device
Changed lines of the file:
@@
 EESchema Schematic File Version 4
-LIBS:Nueva carpeta-cache
-EELAYER 26 0
+EELAYER 30 0
 EELAYER END
 $Descr A4 11693 8268
@@
 	10700 1000 10700 500
 $Comp
-L atmel:ATMEGA328P-PU U1
+L Nueva-carpeta-rescue:ATMEGA328P-PU-atmel U1
 U 1 1 5DC597F1
 P 2850 2150
@@
 $EndComp
 $Comp
-L device:R R1
+L Nueva-carpeta-rescue:R-device R1
 U 1 1 5DC598B6
 P 4350 2350
@@
 $EndComp
 $Comp
-L device:Crystal Y1
+L Nueva-carpeta-rescue:Crystal-device Y1
 U 1 1 5DC599ED
 P 1200 2000
@@
 $EndComp
 $Comp
-L device:C C2
+L Nueva-carpeta-rescue:C-device C2
 U 1 1 5DC59A92
 P 1600 2300
@@
 $EndComp
 $Comp
-L device:C C1
+L Nueva-carpeta-rescue:C-device C1
 U 1 1 5DC59B4B
 P 850 2300
@@
 10(**/SS)
 $Comp
-L device:R R2
+L Nueva-carpeta-rescue:R-device R2
 U 1 1 5DC59958
 P 950 5000
@@
 $EndComp
 $Comp
-L device:LED_ALT D1
+L Nueva-carpeta-rescue:LED_ALT-device D1
 U 1 1 5DC6D160
 P 950 4600
@@
 	950  5150 950  5250
 $Comp
-L device:R R3
+L Nueva-carpeta-rescue:R-device R3
 U 1 1 5DC718A3
 P 1550 4600
@@
 $EndComp
 $Comp
-L device:LED_ALT D2
+L Nueva-carpeta-rescue:LED_ALT-device D2
 U 1 1 5DC718A9
 P 1550 5000
@@
 	1550 5150 1550 5250
 $Comp
-L device:R R4
+L Nueva-carpeta-rescue:R-device R4
 U 1 1 5DC7306A
 P 2200 4600
@@
 $EndComp
 $Comp
-L device:LED_ALT D3
+L Nueva-carpeta-rescue:LED_ALT-device D3
 U 1 1 5DC73070
 P 2200 5000
@@
 	2200 5150 2200 5250
 $Comp
-L device:R R5
+L Nueva-carpeta-rescue:R-device R5
 U 1 1 5DC748DE
 P 2650 4600
@@
 $EndComp
 $Comp
-L device:LED_ALT D4
+L Nueva-carpeta-rescue:LED_ALT-device D4
 U 1 1 5DC748E4
 P 2650 5000
@@
 	1550 4350 1550 4450
 $Comp
-L device:R R6
+L Nueva-carpeta-rescue:R-device R6
 U 1 1 5DC7B925
 P 3100 4600
@@
 $EndComp
 $Comp
-L device:LED_ALT D5
+L Nueva-carpeta-rescue:LED_ALT-device D5
 U 1 1 5DC7B92B
 P 3100 5000
